File: solenoid-1.kicad_sch (KiCad schematic)
At the start: 32 parts, among them J1 SIGNAL, J2 Solenoid Terminal, Q1 IRLZ44N, U1 PC817, U2 USBC - PD - 20V, U3 LM7812, U4 NE555

Commit message: added input LED resistor
Parts:
- added R1: 470, symbol Device:R_Small
- C9: value 1000uF 35V -> 1000uF 50V (35V min)
- renumbered R9 to R10, R10 to R11, R1 to R2, R2 to R3, R3 to R4, R4 to R5, R5 to R6, R6 to R7, R7 to R8, R8 to R9
Connections:
- net at J1.1 (Pin_1): now also R1.1; no longer U1.1
- new net: R1.2, U1.1
Other:
- moved on the sheet: J1
Changed lines of the file:
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@@
 		(rev "11")
 		(company "Leon Springs Baptist Church AWANA Program")
-		(comment 1 "Signal 3V - 12V ( Isolated via Optocoupler )")
+		(comment 1 "Signal 9V Battery (3V-12V) ( Isolated via Optocoupler )")
 		(comment 2 "Relay Timer Trimmer: 50ms - 5.2s")
 		(comment 3 "USBC Power 65W ( Min 45W ) ")
@@
 	)
 	(junction
-		(at 41.91 151.13)
-		(diameter 0)
-		(color 0 0 0 0)
-	)
-	(junction
 		(at 41.91 140.97)
 		(diameter 0)
@@
 	(wire
 		(pts
-			(xy 41.91 151.13) (xy 44.45 151.13)
-		)
-		(stroke
-			(width 0)
-			(type default)
-		)
-	)
-	(wire
-		(pts
 			(xy 113.03 46.99) (xy 130.81 46.99)
 		)
@@
 	(wire
 		(pts
-			(xy 25.4 140.97) (xy 25.4 142.24)
+			(xy 21.59 140.97) (xy 21.59 142.24)
 		)
 		(stroke
@@
 	(wire
 		(pts
-			(xy 26.67 146.05) (xy 25.4 146.05)
-		)
-		(stroke
-			(width 0)
-			(type default)
-		)
-	)
-	(wire
-		(pts
-			(xy 41.91 151.13) (xy 41.91 147.32)
+			(xy 26.67 146.05) (xy 21.59 146.05)
 		)
 		(stroke
@@
 	(wire
 		(pts
-			(xy 26.67 140.97) (xy 25.4 140.97)
-		)
-		(stroke
-			(width 0)
-			(type default)
-		)
-	)
-	(wire
-		(pts
 			(xy 41.91 124.46) (xy 41.91 119.38)
 		)
@@
 	(wire
 		(pts
-			(xy 25.4 146.05) (xy 25.4 144.78)
+			(xy 21.59 146.05) (xy 21.59 144.78)
 		)
 		(stroke
@@
 		(dnp no)
 		(fields_autoplaced yes)
-		(property "Reference" "R9"
+		(property "Reference" "R10"
 			(at 110.49 67.31 90)
 			(effects
@@
 			(project ""
 				(path "/0c404785-1fe3-436f-9caa-e515805d096a"
-					(reference "R9")
+					(reference "R10")
 					(unit 1)
 				)
@@
 		(on_board yes)
 		(dnp no)
-		(property "Reference" "R6"
+		(property "Reference" "R7"
 			(at 67.31 125.7299 0)
 			(effects
@@
 			(project ""
 				(path "/0c404785-1fe3-436f-9caa-e515805d096a"
-					(reference "R6")
+					(reference "R7")
 					(unit 1)
 				)
@@
 		(on_board yes)
 		(dnp no)
-		(property "Reference" "R10"
+		(property "Reference" "R11"
 			(at 123.19 139.6999 0)
 			(effects
@@
 			(project ""
 				(path "/0c404785-1fe3-436f-9caa-e515805d096a"
-					(reference "R10")
+					(reference "R11")
 					(unit 1)
 				)
@@
 		(on_board yes)
 		(dnp no)
-		(property "Reference" "R2"
+		(property "Reference" "R3"
 			(at 54.61 133.3499 0)
 			(effects
@@
 			(project ""
 				(path "/0c404785-1fe3-436f-9caa-e515805d096a"
-					(reference "R2")
+					(reference "R3")
 					(unit 1)
 				)
@@
 		(on_board yes)
 		(dnp no)
-		(property "Reference" "R8"
+		(property "Reference" "R9"
 			(at 106.68 138.43 90)
 			(effects
@@
 			(project ""
 				(path "/0c404785-1fe3-436f-9caa-e515805d096a"
-					(reference "R8")
+					(reference "R9")
 					(unit 1)
 				)
@@
 	)
 	(symbol
+		(lib_id "Device:R_Small")
+		(at 24.13 140.97 90)
+		(unit 1)
+		(exclude_from_sim no)
+		(in_bom yes)
+		(on_board yes)
+		(dnp no)
+		(fields_autoplaced yes)
+		(property "Reference" "R1"
+			(at 24.13 135.89 90)
+			(effects
+				(font
+					(size 1.016 1.016)
+				)
+			)
+		)
+		(property "Value" "470"
+			(at 24.13 138.43 90)
+			(effects
+				(font
+					(size 1.27 1.27)
+				)
+			)
+		)
+		(property "Footprint" ""
+			(at 24.13 140.97 0)
+			(effects
+				(font
+					(size 1.27 1.27)
+				)
+				(hide yes)
+			)
+		)
+		(property "Datasheet" "~"
+			(at 24.13 140.97 0)
+			(effects
+				(font
+					(size 1.27 1.27)
+				)
+				(hide yes)
+			)
+		)
+		(property "Description" "Resistor, small symbol"
+			(at 24.13 140.97 0)
+			(effects
+				(font
+					(size 1.27 1.27)
+				)
+				(hide yes)
+			)
+		)
+		(pin "2"
+		)
+		(pin "1"
+		)
+		(instances
+			(project ""
+				(path "/0c404785-1fe3-436f-9caa-e515805d096a"
+					(reference "R1")
+					(unit 1)
+				)
+			)
+		)
+	)
+	(symbol
 		(lib_id "Device:C_Small")
 		(at 44.45 100.33 0)
@@
 			)
 		)
-		(property "Value" "1000uF 35V"
+		(property "Value" "1000uF 50V (35V min)"
 			(at 118.491 39.37 90)
 			(effects
@@
 	(symbol
 		(lib_id "Connector:Screw_Terminal_01x02")
-		(at 20.32 142.24 0)
+		(at 16.51 142.24 0)
 		(mirror y)
 		(unit 1)
@@
 		(fields_autoplaced yes)
 		(property "Reference" "J1"
-			(at 20.32 135.89 0)
+			(at 16.51 135.89 0)
 			(effects
 				(font
@@
 		)
 		(property "Value" "SIGNAL"
-			(at 20.32 138.43 0)
+			(at 16.51 138.43 0)
 			(effects
 				(font
@@
 		)
 		(property "Footprint" ""
-			(at 20.32 142.24 0)
+			(at 16.51 142.24 0)
 			(effects
 				(font
@@
 		)
 		(property "Datasheet" "~"
-			(at 20.32 142.24 0)
+			(at 16.51 142.24 0)
 			(effects
 				(font
@@
 		)
 		(property "Description" "Generic screw terminal, single row, 01x02, script generated (kicad-library-utils/schlib/autogen/connector/)"
-			(at 20.32 142.24 0)
+			(at 16.51 142.24 0)
 			(effects
 				(font
@@
 		)
 		(property "Vendor Link" ""
-			(at 20.32 142.24 0)
+			(at 16.51 142.24 0)
 			(effects
 				(font
@@
 		)
 		(property "Vendor Summary" ""
-			(at 20.32 142.24 0)
+			(at 16.51 142.24 0)
 			(effects
 				(font
@@
 		(on_board yes)
 		(dnp no)
-		(property "Reference" "R1"
+		(property "Reference" "R2"
 			(at 39.37 115.5699 0)
 			(effects
@@
 			(project ""
 				(path "/0c404785-1fe3-436f-9caa-e515805d096a"
-					(reference "R1")
+					(reference "R2")
 					(unit 1)
 				)
@@
 		(dnp no)
 		(fields_autoplaced yes)
-		(property "Reference" "R3"
+		(property "Reference" "R4"
 			(at 62.23 133.3499 0)
 			(effects
@@
 			(project ""
 				(path "/0c404785-1fe3-436f-9caa-e515805d096a"
-					(reference "R3")
+					(reference "R4")
 					(unit 1)
 				)
@@
 		(on_board yes)
 		(dnp no)
-		(property "Reference" "R5"
+		(property "Reference" "R6"
 			(at 66.04 118.1099 0)
 			(effects
@@
 			(project ""
 				(path "/0c404785-1fe3-436f-9caa-e515805d096a"
-					(reference "R5")
+					(reference "R6")
 					(unit 1)
 				)
@@
 		(on_board yes)
 		(dnp no)
-		(property "Reference" "R4"
+		(property "Reference" "R5"
 			(at 66.04 147.32 90)
 			(effects
@@
 			(project ""
 				(path "/0c404785-1fe3-436f-9caa-e515805d096a"
-					(reference "R4")
+					(reference "R5")
 					(unit 1)
 				)
@@
 		(dnp no)
 		(fields_autoplaced yes)
-		(property "Reference" "R7"
+		(property "Reference" "R8"
 			(at 76.2 92.7099 0)
 			(effects
@@
 			(project ""
 				(path "/0c404785-1fe3-436f-9caa-e515805d096a"
-					(reference "R7")
+					(reference "R8")
 					(unit 1)
 				)
