File: solenoid-1.kicad_sch (KiCad schematic)
At the start: 33 parts, among them J1 SIGNAL, J2 Solenoid Terminal, Q1 IRLZ44N, U1 PC817, U2 USBC - PD - 20V, U3 LM7812, U4 NE555

Commit message: upd
Connections:
- net +12V: no longer R2.1
- net at C1.2, C2.2, C4.2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: now also LED1.1 (K), R2.1
- net at C3.2, R3.2, U1.4: no longer LED1.1 (K)
Other:
- moved on the sheet: C3, J1, LED1, R1, R2, R3, R4, U1

Commit message: v15
Parts:
- removed LED2: GREEN VF 3.2 IF 20mA, LED_THT:LED_D3.0mm_IRBlack, symbol LED:TSAL4400
- removed R8: 470, symbol Device:R_Small
- C5: value 47uF -> 4.7uF
- C8: value 100nF -> 0.1uF
- LED1: value BLUE VF 3.2 IF 20mA -> RED VF 2.1 IF 20mA
- LED2: renamed from LED3; value ORANGE VF1.2 IF 20mA -> ORANGE VF2.1 IF 20mA
- R1: value 470 -> 1K
- R10: renamed from R11; value 10K -> 47K
- R6: value 100K (RM065) -> 1M (RM065)
- R7: value 1K -> 100K
- R9: renamed from R10; value 680 -> 470
- renumbered R9 to R8
